Commit message: minor bug fix

File: assets/three_link_planar.urdf (robot description, URDF)
Before this commit: robot three_link_robot, 3 links, 3 joints
Links:
- added link base_link
- link link1: geometry collision box size=1 0.05 0.05; visual box size=1 0.05 0.05
- link link2: geometry collision box size=1 0.05 0.05; visual box size=1 0.05 0.05
- link link3: geometry collision box size=1 0.05 0.05; visual box size=1 0.05 0.05
Joints:
- joint joint1: limit lower=-1.57 upper=1.57 effort=10.0 velocity=2.0 -> lower=-3.14159 upper=3.14159 effort=100 velocity=100; parent world -> base_link
- joint joint2: limit lower=0 upper=3.14 effort=10.0 velocity=2.0 -> lower=-3.14159 upper=3.14159 effort=100 velocity=100; origin xyz=1.0 0 0 rpy=0 0 0 -> xyz=1 0 0 rpy=0 0 0
- joint joint3: limit lower=-2.36 upper=2.36 effort=10.0 velocity=2.0 -> lower=-3.14159 upper=3.14159 effort=100 velocity=100; origin xyz=1.0 0 0 rpy=0 0 0 -> xyz=1 0 0 rpy=0 0 0
